Commit message: Improved the base model a bit

File: resources/urdfs/pg70.urdf (robot description, URDF)
Before this commit: robot schunk_pg70, 8 links, 7 joints
Links:
- link pg70_base_link: geometry collision mesh filename=package://manos_description/meshes/schunk_pg70/pg70.dae; visual mesh filename=package://manos_description/meshes/schunk_pg70/pg70.dae

Commit message: Improved the overall accuracy of the model, based on the new mesh file for the gripper

File: resources/urdfs/pg70.urdf (robot description, URDF)
Before this commit: robot schunk_pg70, 8 links, 7 joints
Links:
- link gripper_power_cable: geometry collision box size=0.012 0.012 0.035; visual box size=0.012 0.012 0.035
Joints:
- joint gripper_power_cable_joint: origin xyz=-0.011 -0.011 0.011 rpy=0 0 1.57079632679 -> xyz=-0.011 -0.021 0.031 rpy=0 0 1.57079632679
- joint gripper_power_joint: origin xyz=0.004 0.03 0.08 rpy=0 1.57079632679 0 -> xyz=0 -0.015 0.08 rpy=0 1.57079632679 0
- joint pg70_finger1_joint: origin xyz=0 0.0765 0.04 rpy=0 0 0 -> xyz=0 0.0475 0.04 rpy=0 0 0
- joint pg70_finger2_joint: origin xyz=0 0.0765 -0.04 rpy=0 0 0 -> xyz=0 0.0475 -0.04 rpy=0 0 0
